Commit message: basic position tracking

File: model/urdf/GEN3_URDF_V12.urdf (robot description, URDF)
Before this commit: robot GEN3_URDF_V12, 9 links, 8 joints
Links:
- removed link EndEffector_Link
- added link end_effector_link
Joints:
- joint EndEffector: child EndEffector_Link -> end_effector_link
