Commit message: add rudimentary end-effector contact model

File: models/hande_gripper/urdf/robotiq_hande_static.urdf (robot description, URDF)
Before this commit: robot robotiq_hande, 3 links, 2 joints
Links:
- removed link hande_robotiq_hande_base_link
- added link hande_base_link, mass 0.86387; collision cylinder length=0.092 radius=0.038; visual mesh filename=../meshes/hand-e.obj scale=0.001 0.001 0.001
- link hande_left_finger: geometry collision box size=0.007 0.02 0.02; visual mesh filename=../meshes/finger_1.obj scale=0.001 0.001 0.001
- link hande_right_finger: geometry collision box size=0.007 0.02 0.02; visual mesh filename=../meshes/finger_2.obj scale=0.001 0.001 0.001
Joints:
- joint hande_joint_left_finger: parent hande_robotiq_hande_base_link -> hande_base_link
- joint hande_joint_right_finger: parent hande_robotiq_hande_base_link -> hande_base_link
