Commit message: extend gripper collision surface all the way to base of gripper

File: models/hande_gripper/urdf/robotiq_hande.urdf (robot description, URDF)
Before this commit: robot robotiq_hande, 3 links, 2 joints
Links:
- link hande_left_finger: geometry collision box size=0.007 0.02 0.045; visual mesh filename=../meshes/finger_1.obj scale=0.001 0.001 0.001
- link hande_right_finger: geometry collision box size=0.007 0.02 0.045; visual mesh filename=../meshes/finger_2.obj scale=0.001 0.001 0.001

File: models/hande_gripper/urdf/robotiq_hande_static.urdf (robot description, URDF)
Before this commit: robot robotiq_hande, 3 links, 2 joints
Links:
- link hande_left_finger: geometry collision box size=0.007 0.02 0.045; visual mesh filename=../meshes/finger_1.obj scale=0.001 0.001 0.001
- link hande_right_finger: geometry collision box size=0.007 0.02 0.045; visual mesh filename=../meshes/finger_2.obj scale=0.001 0.001 0.001
