Commit message: preliminary use of meshcat for visualization

File: models/2f_85_gripper/urdf/robotiq_2f_85.urdf (robot description, URDF)
Before this commit: robot robotiq_arg2f_85_model, 11 links, 10 joints
Links:
- link left_inner_finger: mass None -> 0.0104003125914103
- link left_inner_knuckle: mass None -> 0.0271177346495152; geometry visual mesh filename=../meshes/visual/robotiq_arg2f_85_inner_knuckle.obj scale=0.001 0.001 0.001
- link left_outer_finger: mass None -> 0.022614240507152
- link left_outer_knuckle: mass None -> 0.00853198276973456
- link right_inner_finger: mass None -> 0.0104003125914103
- link right_inner_knuckle: mass None -> 0.0271177346495152; geometry visual mesh filename=../meshes/visual/robotiq_arg2f_85_inner_knuckle.obj scale=0.001 0.001 0.001
- link right_outer_finger: mass None -> 0.022614240507152
- link right_outer_knuckle: mass None -> 0.00853198276973456

Commit message: increase bushing stiffness

File: models/2f_85_gripper/urdf/robotiq_2f_85.urdf (robot description, URDF)
Before this commit: robot robotiq_arg2f_85_model, 11 links, 10 joints
Joints:
- joint left_inner_knuckle_joint: limit lower=0 upper=0.8757 effort=1000 velocity=2.0 -> lower=0 upper=0.8 effort=1000 velocity=2.0
- joint right_inner_knuckle_joint: limit lower=0 upper=0.8757 effort=1000 velocity=2.0 -> lower=0 upper=0.8 effort=1000 velocity=2.0

Commit message: open position looks good

File: models/2f_85_gripper/urdf/robotiq_2f_85.urdf (robot description, URDF)
Before this commit: robot robotiq_arg2f_85_model, 11 links, 10 joints
Joints:
- joint left_inner_knuckle_joint: limit lower=0 upper=0.8 effort=1000 velocity=2.0 -> lower=0 upper=0.8757 effort=1000 velocity=2.0
- joint right_inner_knuckle_joint: limit lower=0 upper=0.8 effort=1000 velocity=2.0 -> lower=0 upper=0.8757 effort=1000 velocity=2.0
