Commit message: include camera in 7DoF simulation model

File: models/gen3_7dof/urdf/GEN3_URDF_V12.urdf (robot description, URDF)
Before this commit: robot GEN3_URDF_V12, 9 links, 8 joints
Links:
- removed link bracelet_no_vision_link
- added link bracelet_with_vision_link, mass 0.5006; collision mesh filename=../meshes/bracelet_with_vision_link.obj; visual mesh filename=../meshes/bracelet_with_vision_link.obj
Joints:
- joint Actuator7: child bracelet_no_vision_link -> bracelet_with_vision_link
- joint EndEffector: parent bracelet_no_vision_link -> bracelet_with_vision_link
